File: USB_to_UART.kicad_sch (KiCad schematic)
At the start: 13 parts, among them J1 USB_B_Micro, U1 FT230XS

Commit message: changes to schematic and PCB
Parts:
- added D1, D2: LED, LED_SMD:LED_0805_2012Metric, symbol Device:LED
- C1, C2, C3, C4: footprint (none) -> Capacitor_SMD:C_0805_2012Metric
- FB1: footprint (none) -> Inductor_SMD:L_0805_2012Metric
- J1: footprint (none) -> Connector_USB:USB_Micro-B_Wuerth_629105150521
- R1, R2, R3, R4: footprint (none) -> Resistor_SMD:R_0805_2012Metric
- TP1, TP2: footprint (none) -> TestPoint:TestPoint_Plated_Hole_D2.0mm
Connections:
- net USB_3V3: now also D1.2 (A), D2.2 (A); no longer R3.1, R4.1
- net UART_RXD renamed UART1_Rx
- net UART_TXD renamed UART1_Tx
- new net: D1.1 (K), R3.1
- new net: D2.1 (K), R4.1
Other:
- moved on the sheet: C1, C2, C3, C4, FB1, J1, R1, R2, R3, R4, TP1, TP2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

Commit message: changed schematics
Parts:
- added C39: 4.7 uF, Capacitor_SMD:C_0805_2012Metric, symbol Device:C
- added C40: 100 nF, Capacitor_SMD:C_0805_2012Metric, symbol Device:C
- C1: value 4.7 pF -> 100 nF
- R3, R4: value 470 -> 750
- TP1, TP2: footprint TestPoint:TestPoint_Plated_Hole_D2.0mm -> TestPoint:TestPoint_Pad_2.0x2.0mm
Connections:
- net Earth: now also C39.2, C40.2
- net VBUS: now also C39.1, C40.1
